File: pamp.sch (KiCad schematic (older format))
At the start: 49 parts, among them U1 NE5532, U2 OPA1612AxD, U3 NE5532, U4 OPA1612AxD, U5 NE5532, U6 NE5532

Commit message: Update.
Signed-off-by: Nenad Radulovic <nenad.b.radulovic@gmail.com>
Parts:
- added R17, R18, R19, R20: 10k, Resistor_SMD:R_1206_3216Metric_Pad1.42x1.75mm_HandSolder, symbol Device:R
- R15, R16: value 20k -> 10k
- renumbered R17 to R21, R18 to R22, R19 to R23, R20 to R24
Connections:
- net at U3.1, U3.2 (-): now also RV1.6; no longer RV1.4
- net at R10.1, R12.2, U3.7: now also RV1.4; no longer RV1.6
- net at R21.2, U2.1: now also R17.1; no longer U2.2 (-)
- net at R22.2, U2.7: now also R18.1; no longer U2.6 (-)
- net at R23.2, U4.1: now also R19.1; no longer U4.2 (-)
- net at R24.2, U4.7: now also R20.1; no longer U4.6 (-)
- new net: R17.2, U2.2 (-)
- new net: R18.2, U2.6 (-)
- new net: R19.2, U4.2 (-)
- new net: R20.2, U4.6 (-)
Changed lines of the file:
@@
 EESchema Schematic File Version 4
+LIBS:picowire-cache
 EELAYER 26 0
 EELAYER END
@@
 encoding utf-8
 Sheet 2 3
-Title ""
-Date ""
-Rev ""
-Comp ""
-Comment1 ""
+Title "PicoWire"
+Date "2018-10-17"
+Rev "1"
+Comp "REAL-TIME CONSULTING"
+Comment1 "Headphone amplifier"
 Comment2 ""
 Comment3 ""
@@
 $EndComp
 $Comp
-L power:GNDA #PWR09
+L power:GNDA #PWR05
 U 1 1 5BCA25D6
 P 1700 2900
-F 0 "#PWR09" H 1700 2650 50  0001 C CNN
+F 0 "#PWR05" H 1700 2650 50  0001 C CNN
 F 1 "GNDA" H 1705 2727 50  0000 C CNN
 F 2 "" H 1700 2900 50  0001 C CNN
@@
 $EndComp
 $Comp
-L power:GNDA #PWR010
+L power:GNDA #PWR06
 U 1 1 5BCA48A3
 P 1700 4200
-F 0 "#PWR010" H 1700 3950 50  0001 C CNN
+F 0 "#PWR06" H 1700 3950 50  0001 C CNN
 F 1 "GNDA" H 1705 4027 50  0000 C CNN
 F 2 "" H 1700 4200 50  0001 C CNN
@@
 Wire Wire Line
 	1200 3600 1300 3600
-Wire Wire Line
-	4000 2950 4500 2950
-Wire Wire Line
-	4000 3700 4000 3150
-Wire Wire Line
-	4000 3150 4500 3150
 $Comp
 L Amplifier_Operational:NE5532 U5
@@
 Connection ~ 5900 2400
 $Comp
-L power:GNDA #PWR011
+L power:GNDA #PWR07
 U 1 1 5BCB55C2
 P 6300 3000
-F 0 "#PWR011" H 6300 2750 50  0001 C CNN
+F 0 "#PWR07" H 6300 2750 50  0001 C CNN
 F 1 "GNDA" V 6305 2873 50  0000 R CNN
 F 2 "" H 6300 3000 50  0001 C CNN
@@
 	9200 1700 9200 1900
 Wire Wire Line
-	9200 1900 10000 1900
-Wire Wire Line
 	10000 1900 10000 1600
 Wire Wire Line
@@
 	9200 2800 9200 3000
 Wire Wire Line
-	9200 3000 10000 3000
-Wire Wire Line
 	10000 3000 10000 2700
 Wire Wire Line
 	10000 2700 9900 2700
 $Comp
-L Device:R R17
+L Device:R R21
 U 1 1 5BCBDA47
 P 10250 1600
-F 0 "R17" V 10043 1600 50  0000 C CNN
+F 0 "R21" V 10043 1600 50  0000 C CNN
 F 1 "10" V 10134 1600 50  0000 C CNN
 F 2 "Resistor_SMD:R_1206_3216Metric_Pad1.42x1.75mm_HandSolder" V 10180 1600 50  0001 C CNN
@@
 $EndComp
 $Comp
-L Device:R R18
+L Device:R R22
 U 1 1 5BCBDA4E
 P 10250 2700
-F 0 "R18" V 10043 2700 50  0000 C CNN
+F 0 "R22" V 10043 2700 50  0000 C CNN
 F 1 "10" V 10134 2700 50  0000 C CNN
 F 2 "Resistor_SMD:R_1206_3216Metric_Pad1.42x1.75mm_HandSolder" V 10180 2700 50  0001 C CNN
@@
 Wire Wire Line
 	7200 4200 7200 4700
-Wire Wire Line
-	7200 4700 4500 4700
-Wire Wire Line
-	4500 4700 4500 3450
 Connection ~ 7200 4200
 Wire Wire Line
@@
 	9200 3700 9200 3900
 Wire Wire Line
-	9200 3900 10000 3900
-Wire Wire Line
 	10000 3900 10000 3600
 Wire Wire Line
@@
 	9200 4800 9200 5000
 Wire Wire Line
-	9200 5000 10000 5000
-Wire Wire Line
 	10000 5000 10000 4700
 Wire Wire Line
 	10000 4700 9900 4700
 $Comp
-L Device:R R19
+L Device:R R23
 U 1 1 5BCF864A
 P 10250 3600
-F 0 "R19" V 10043 3600 50  0000 C CNN
+F 0 "R23" V 10043 3600 50  0000 C CNN
 F 1 "10" V 10134 3600 50  0000 C CNN
 F 2 "Resistor_SMD:R_1206_3216Metric_Pad1.42x1.75mm_HandSolder" V 10180 3600 50  0001 C CNN
@@
 $EndComp
 $Comp
-L Device:R R20
+L Device:R R24
 U 1 1 5BCF8651
 P 10250 4700
-F 0 "R20" V 10043 4700 50  0000 C CNN
+F 0 "R24" V 10043 4700 50  0000 C CNN
 F 1 "10" V 10134 4700 50  0000 C CNN
 F 2 "Resistor_SMD:R_1206_3216Metric_Pad1.42x1.75mm_HandSolder" V 10180 4700 50  0001 C CNN
@@
 	7200 2500 7300 2500
 $Comp
-L power:GNDA #PWR012
+L power:GNDA #PWR08
 U 1 1 5BD08110
 P 7600 3000
-F 0 "#PWR012" H 7600 2750 50  0001 C CNN
+F 0 "#PWR08" H 7600 2750 50  0001 C CNN
 F 1 "GNDA" V 7605 2873 50  0000 R CNN
 F 2 "" H 7600 3000 50  0001 C CNN
@@
 P 8750 4600
 F 0 "R16" V 8543 4600 50  0000 C CNN
-F 1 "20k" V 8634 4600 50  0000 C CNN
+F 1 "10k" V 8634 4600 50  0000 C CNN
 F 2 "Resistor_SMD:R_1206_3216Metric_Pad1.42x1.75mm_HandSolder" V 8680 4600 50  0001 C CNN
 F 3 "~" H 8750 4600 50  0001 C CNN
@@
 $EndComp
 $Comp
-L power:GNDA #PWR014
+L power:GNDA #PWR010
 U 1 1 5BD330B6
 P 8500 4600
-F 0 "#PWR014" H 8500 4350 50  0001 C CNN
+F 0 "#PWR010" H 8500 4350 50  0001 C CNN
 F 1 "GNDA" V 8505 4473 50  0000 R CNN
 F 2 "" H 8500 4600 50  0001 C CNN
@@
 P 8750 1500
 F 0 "R15" V 8543 1500 50  0000 C CNN
-F 1 "20k" V 8634 1500 50  0000 C CNN
+F 1 "10k" V 8634 1500 50  0000 C CNN
 F 2 "Resistor_SMD:R_1206_3216Metric_Pad1.42x1.75mm_HandSolder" V 8680 1500 50  0001 C CNN
 F 3 "~" H 8750 1500 50  0001 C CNN
@@
 $EndComp
 $Comp
-L power:GNDA #PWR013
+L power:GNDA #PWR09
 U 1 1 5BD3316B
 P 8500 1500
-F 0 "#PWR013" H 8500 1250 50  0001 C CNN
+F 0 "#PWR09" H 8500 1250 50  0001 C CNN
 F 1 "GNDA" V 8505 1373 50  0000 R CNN
 F 2 "" H 8500 1500 50  0001 C CNN
@@
 $EndComp
 $Comp
-L power:GNDA #PWR04
+L power:GNDA #PWR03
 U 1 1 5BDC821F
 P 1000 5500
-F 0 "#PWR04" H 1000 5250 50  0001 C CNN
+F 0 "#PWR03" H 1000 5250 50  0001 C CNN
 F 1 "GNDA" V 1005 5373 50  0000 R CNN
 F 2 "" H 1000 5500 50  0001 C CNN
@@
 $EndComp
 $Comp
-L power:GNDA #PWR07
+L power:GNDA #PWR04
 U 1 1 5BEA9D51
 P 1000 7000
-F 0 "#PWR07" H 1000 6750 50  0001 C CNN
+F 0 "#PWR04" H 1000 6750 50  0001 C CNN
 F 1 "GNDA" V 1005 6873 50  0000 R CNN
 F 2 "" H 1000 7000 50  0001 C CNN
@@
 Text GLabel 1000 7500 0    50   Input ~ 0
 VEE
+$Comp
+L Device:R R17
+U 1 1 5C0B3D52
+P 9750 1900
+F 0 "R17" V 9865 1900 50  0000 C CNN
+F 1 "10k" V 9956 1900 50  0000 C CNN
+F 2 "Resistor_SMD:R_1206_3216Metric_Pad1.42x1.75mm_HandSolder" V 9680 1900 50  0001 C CNN
+F 3 "~" H 9750 1900 50  0001 C CNN
+	1    9750 1900
+	0    1    1    0
+$EndComp
+$Comp
+L Device:R R18
+U 1 1 5C0B3DEA
+P 9750 3000
+F 0 "R18" V 9865 3000 50  0000 C CNN
+F 1 "10k" V 9956 3000 50  0000 C CNN
+F 2 "Resistor_SMD:R_1206_3216Metric_Pad1.42x1.75mm_HandSolder" V 9680 3000 50  0001 C CNN
+F 3 "~" H 9750 3000 50  0001 C CNN
+	1    9750 3000
+	0    1    1    0
+$EndComp
+$Comp
+L Device:R R19
+U 1 1 5C0B3E78
+P 9750 3900
+F 0 "R19" V 9865 3900 50  0000 C CNN
+F 1 "10k" V 9956 3900 50  0000 C CNN
+F 2 "Resistor_SMD:R_1206_3216Metric_Pad1.42x1.75mm_HandSolder" V 9680 3900 50  0001 C CNN
+F 3 "~" H 9750 3900 50  0001 C CNN
+	1    9750 3900
+	0    1    1    0
+$EndComp
+$Comp
+L Device:R R20
+U 1 1 5C0B3F14
+P 9750 5000
+F 0 "R20" V 9865 5000 50  0000 C CNN
+F 1 "10k" V 9956 5000 50  0000 C CNN
+F 2 "Resistor_SMD:R_1206_3216Metric_Pad1.42x1.75mm_HandSolder" V 9680 5000 50  0001 C CNN
+F 3 "~" H 9750 5000 50  0001 C CNN
+	1    9750 5000
+	0    1    1    0
+$EndComp
+Wire Wire Line
+	9600 1900 9200 1900
+Wire Wire Line
+	9900 1900 10000 1900
+Wire Wire Line
+	9900 3000 10000 3000
+Wire Wire Line
+	9600 3000 9200 3000
+Wire Wire Line
+	9600 3900 9200 3900
+Wire Wire Line
+	9900 3900 10000 3900
+Wire Wire Line
+	9900 5000 10000 5000
+Wire Wire Line
+	9600 5000 9200 5000
+Wire Wire Line
+	4500 3150 4300 3150
+Wire Wire Line
+	4300 3150 4300 4700
+Wire Wire Line
+	4300 4700 7200 4700
+Wire Wire Line
+	4500 3450 4500 3700
+Wire Wire Line
+	4500 3700 4000 3700
+Wire Wire Line
+	4000 2950 4500 2950
 $EndSCHEMATC
