File: psupply.sch (KiCad schematic (older format))
At the start: 23 parts, among them Q1 BDX53, U7 OPA1688, U8 OPA1688, U9 OPA1688

Commit message: Update.
Signed-off-by: Nenad Radulovic <nenad.b.radulovic@gmail.com>
Parts:
- renumbered R21 to R25, R22 to R26, R23 to R27, R24 to R28, R25 to R29, R26 to R30, R27 to R31, R28 to R32, R29 to R33
Changed lines of the file:
@@
 EESchema Schematic File Version 4
+LIBS:picowire-cache
 EELAYER 26 0
 EELAYER END
@@
 encoding utf-8
 Sheet 3 3
-Title ""
-Date ""
-Rev ""
-Comp ""
-Comment1 ""
+Title "PicoWire"
+Date "2018-10-17"
+Rev "1"
+Comp "REAL-TIME CONSULTING"
+Comment1 "Headphone amplifier"
 Comment2 ""
 Comment3 ""
@@
 $EndComp
 $Comp
-L Device:R R21
+L Device:R R25
 U 1 1 5BC3B20B
 P 3000 1750
-F 0 "R21" H 3070 1796 50  0000 L CNN
+F 0 "R25" H 3070 1796 50  0000 L CNN
 F 1 "1k" H 3070 1705 50  0000 L CNN
 F 2 "Resistor_SMD:R_1206_3216Metric_Pad1.42x1.75mm_HandSolder" V 2930 1750 50  0001 C CNN
@@
 	8200 4600 8200 3700
 $Comp
-L Device:R R24
+L Device:R R28
 U 1 1 5BC3E475
 P 9450 1200
-F 0 "R24" V 9243 1200 50  0000 C CNN
+F 0 "R28" V 9243 1200 50  0000 C CNN
 F 1 "10" V 9334 1200 50  0000 C CNN
 F 2 "Resistor_SMD:R_1206_3216Metric_Pad1.42x1.75mm_HandSolder" V 9380 1200 50  0001 C CNN
@@
 	9700 4700 9700 3800
 $Comp
-L power:GNDA #PWR022
+L power:GNDA #PWR014
 U 1 1 5BC45CAC
 P 9700 6100
-F 0 "#PWR022" H 9700 5850 50  0001 C CNN
+F 0 "#PWR014" H 9700 5850 50  0001 C CNN
 F 1 "GNDA" H 9705 5927 50  0000 C CNN
 F 2 "" H 9700 6100 50  0001 C CNN
@@
 Connection ~ 3800 6200
 $Comp
-L Device:R R22
+L Device:R R26
 U 1 1 5BC8AE3D
 P 7700 3450
-F 0 "R22" H 7770 3496 50  0000 L CNN
+F 0 "R26" H 7770 3496 50  0000 L CNN
 F 1 "10k" H 7770 3405 50  0000 L CNN
 F 2 "Resistor_SMD:R_1206_3216Metric_Pad1.42x1.75mm_HandSolder" V 7630 3450 50  0001 C CNN
@@
 $EndComp
 $Comp
-L Device:R R23
+L Device:R R27
 U 1 1 5BC8AE44
 P 7700 3950
-F 0 "R23" H 7770 3996 50  0000 L CNN
+F 0 "R27" H 7770 3996 50  0000 L CNN
 F 1 "10k" H 7770 3905 50  0000 L CNN
 F 2 "Resistor_SMD:R_1206_3216Metric_Pad1.42x1.75mm_HandSolder" V 7630 3950 50  0001 C CNN
@@
 	7700 3200 7700 3300
 $Comp
-L power:VCC #PWR020
+L power:VCC #PWR012
 U 1 1 5BC8AE4F
 P 7700 3200
-F 0 "#PWR020" H 7700 3050 50  0001 C CNN
+F 0 "#PWR012" H 7700 3050 50  0001 C CNN
 F 1 "VCC" H 7717 3373 50  0000 C CNN
 F 2 "" H 7700 3200 50  0001 C CNN
@@
 $EndComp
 $Comp
-L power:VEE #PWR021
+L power:VEE #PWR013
 U 1 1 5BC8AE55
 P 7700 4200
-F 0 "#PWR021" H 7700 4050 50  0001 C CNN
+F 0 "#PWR013" H 7700 4050 50  0001 C CNN
 F 1 "VEE" H 7718 4373 50  0000 C CNN
 F 2 "" H 7700 4200 50  0001 C CNN
@@
 $EndComp
 $Comp
-L power:GNDA #PWR019
+L power:GNDA #PWR011
 U 1 1 5BD9F7BC
 P 4600 2000
-F 0 "#PWR019" H 4600 1750 50  0001 C CNN
+F 0 "#PWR011" H 4600 1750 50  0001 C CNN
 F 1 "GNDA" V 4605 1872 50  0000 R CNN
 F 2 "" H 4600 2000 50  0001 C CNN
@@
 $EndComp
 $Comp
-L Device:R R25
+L Device:R R29
 U 1 1 5BDC7193
 P 9450 2000
-F 0 "R25" V 9243 2000 50  0000 C CNN
+F 0 "R29" V 9243 2000 50  0000 C CNN
 F 1 "10" V 9334 2000 50  0000 C CNN
 F 2 "Resistor_SMD:R_1206_3216Metric_Pad1.42x1.75mm_HandSolder" V 9380 2000 50  0001 C CNN
@@
 $EndComp
 $Comp
-L Device:R R26
+L Device:R R30
 U 1 1 5BDC71F5
 P 9450 2900
-F 0 "R26" V 9243 2900 50  0000 C CNN
+F 0 "R30" V 9243 2900 50  0000 C CNN
 F 1 "10" V 9334 2900 50  0000 C CNN
 F 2 "Resistor_SMD:R_1206_3216Metric_Pad1.42x1.75mm_HandSolder" V 9380 2900 50  0001 C CNN
@@
 $EndComp
 $Comp
-L Device:R R27
+L Device:R R31
 U 1 1 5BDC725D
 P 9450 3800
-F 0 "R27" V 9243 3800 50  0000 C CNN
+F 0 "R31" V 9243 3800 50  0000 C CNN
 F 1 "10" V 9334 3800 50  0000 C CNN
 F 2 "Resistor_SMD:R_1206_3216Metric_Pad1.42x1.75mm_HandSolder" V 9380 3800 50  0001 C CNN
@@
 $EndComp
 $Comp
-L Device:R R28
+L Device:R R32
 U 1 1 5BDC72CB
 P 9450 4700
-F 0 "R28" V 9243 4700 50  0000 C CNN
+F 0 "R32" V 9243 4700 50  0000 C CNN
 F 1 "10" V 9334 4700 50  0000 C CNN
 F 2 "Resistor_SMD:R_1206_3216Metric_Pad1.42x1.75mm_HandSolder" V 9380 4700 50  0001 C CNN
@@
 $EndComp
 $Comp
-L Device:R R29
+L Device:R R33
 U 1 1 5BDC7337
 P 9450 5600
-F 0 "R29" V 9243 5600 50  0000 C CNN
+F 0 "R33" V 9243 5600 50  0000 C CNN
 F 1 "10" V 9334 5600 50  0000 C CNN
 F 2 "Resistor_SMD:R_1206_3216Metric_Pad1.42x1.75mm_HandSolder" V 9380 5600 50  0001 C CNN
@@
 VEE
 $Comp
-L power:PWR_FLAG #FLG0101
+L power:PWR_FLAG #FLG01
 U 1 1 5BF4DD8C
 P 4000 1500
-F 0 "#FLG0101" H 4000 1575 50  0001 C CNN
+F 0 "#FLG01" H 4000 1575 50  0001 C CNN
 F 1 "PWR_FLAG" H 4000 1674 50  0000 C CNN
 F 2 "" H 4000 1500 50  0001 C CNN
@@
 $EndComp
 $Comp
-L power:PWR_FLAG #FLG0102
+L power:PWR_FLAG #FLG02
 U 1 1 5BF4F34B
 P 4000 2500
-F 0 "#FLG0102" H 4000 2575 50  0001 C CNN
+F 0 "#FLG02" H 4000 2575 50  0001 C CNN
 F 1 "PWR_FLAG" H 4000 2673 50  0000 C CNN
 F 2 "" H 4000 2500 50  0001 C CNN
@@
 $EndComp
 $Comp
-L power:PWR_FLAG #FLG0103
+L power:PWR_FLAG #FLG03
 U 1 1 5BF4F4F7
 P 9700 5600
-F 0 "#FLG0103" H 9700 5675 50  0001 C CNN
+F 0 "#FLG03" H 9700 5675 50  0001 C CNN
 F 1 "PWR_FLAG" V 9700 5728 50  0000 L CNN
 F 2 "" H 9700 5600 50  0001 C CNN
